File: hardware/hexpansion.kicad_pcb (KiCad board)
At the start: 2 copper layers, 47.1 x 49.9 mm, 50 parts, among them J1 Hexpansion-Connector, J2 Conn_02x03_Odd_Even, J3 OSTVN02A150, J4 OSTVN04A150, J5 Conn_01x02_Pin, Q1 Q_PMOS_DGS, U1 ATTINY85-20SU, U2 BC857BS

Commit message: hardware: update PCB, schematic and gerbers
Sync the revised KiCad board and schematic and the regenerated gerber set
from the latest design.

Co-Authored-By: Claude Opus 4.8 <noreply@anthropic.com>
Parts:
- U2: value BC857BS -> BC857BS-13-F
Connections:
- J1 pad 2: LS_A -> unconnected-(J1-LS_A-Pad2)
- R4 pad 2: GND -> 3V3
- R5 pad 2: GND -> 3V3
Routing:
- net 3V3: track 111.5 -> 114.6 mm
Changed lines of the file:
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@@
 			(drillshape 0)
 			(scaleselection 1)
-			(outputdirectory "nodule-breakout-jan24-gerbers")
+			(outputdirectory "space-unicorn-gerbers")
 		)
 	)
@@
 			(layers "B.Cu" "B.Mask")
 			(roundrect_rratio 0.25)
-			(net "LS_A")
+			(net "unconnected-(J1-LS_A-Pad2)")
 			(pinfunction "LS_A_2")
-			(pintype "bidirectional")
+			(pintype "bidirectional+no_connect")
 		)
 		(pad "3" smd roundrect
@@
 			)
 		)
-		(property "Value" "BC857BS"
+		(property "Value" "BC857BS-13-F"
 			(at 4.6652 -4.1396 0)
 			(layer "F.Fab")
@@
 			(layers "F.Cu" "F.Mask" "F.Paste")
 			(roundrect_rratio 0.25)
-			(net "GND")
+			(net "3V3")
 			(pintype "passive")
 		)
@@
 			(layers "F.Cu" "F.Mask" "F.Paste")
 			(roundrect_rratio 0.25)
-			(net "GND")
+			(net "3V3")
 			(pintype "passive")
 		)
@@
 	)
 	(gr_line
+		(start 127.95 80.15)
+		(end 125.8 81.3)
+		(stroke
+			(width 0.25)
+			(type solid)
+		)
+		(layer "F.Cu")
+		(net "3V3")
+	)
+	(gr_line
+		(start 128.45 81.05)
+		(end 127.45 79.25)
+		(stroke
+			(width 0.25)
+			(type solid)
+		)
+		(layer "F.Cu")
+		(net "3V3")
+	)
+	(gr_line
 		(start 129.175 119.875)
 		(end 127.471449 120.808377)
@@
 	)
 	(segment
+		(start 124.799373 83.570204)
+		(end 124.799373 82.300627)
+		(width 0.25)
+		(layer "F.Cu")
+		(net "3V3")
+	)
+	(segment
 		(start 118.8 96.027604)
 		(end 120.547396 96.027604)
@@
 	)
 	(segment
+		(start 124.799373 83.570204)
+		(end 125.092134 83.277443)
+		(width 0.25)
+		(layer "F.Cu")
+		(net "3V3")
+	)
+	(segment
 		(start 117.5 104.1)
 		(end 117.5 115.596736)
@@
 		(layer "F.Cu")
 		(net "3V3")
+	)
+	(segment
+		(start 124.799373 82.300627)
+		(end 125.8 81.3)
+		(width 0.25)
+		(layer "F.Cu")
+		(net "3V3")
